Commit message: add hand-eye calibration package, done system urdf

File: src/robot_description/urdf/system.urdf.xacro (robot description, xacro)
@@ -1,11 +1,23 @@
 <?xml version="1.0"?>
 <robot name="deep_flip_system" xmlns:xacro="http://ros.org/wiki/xacro">
+  <gazebo>
+    <plugin name="gazebo_ros_control" filename="libgazebo_ros_control.so">
+      <robotNamespace>/</robotNamespace>
+    </plugin>
+  </gazebo>
   <xacro:property name="M_PI" value="3.1415926535"/>
   <!-- UR3 -->
   <xacro:include filename="$(find ur_description)/urdf/ur3.urdf.xacro"/>
+  <!-- Gripper -->
+  <xacro:include filename="$(find robotiq_description)/urdf/robotiq_85_gripper.urdf.xacro" />
+  <!-- Color material -->
   <material name="black">
     <color rgba="0.2 0.2 0.2 1.0"/>
   </material>
+  <material name="green">
+    <color rgba="0.0 1.0 0.0 1.0"/>
+  </material>
   <xacro:ur3_robot prefix="" joint_limited="false"/>
+  <!-- SR300 -->
   <link name="camera_link">
     <visual>
@@ -23,3 +35,34 @@
     <child link="camera_link"/>
   </joint>
+  <!-- Robotiq 2f 85 -->
+  <link name="gripper_root_link"/>
+  <joint name="ee2gripper_joint" type="fixed">
+    <parent link="ee_link"/>
+    <child link="gripper_root_link"/>
+    <origin xyz="0.011 0.0 0.0" rpy="${M_PI} 0.0 0.0"/>
+  </joint>
+  <xacro:robotiq_85_gripper prefix="" parent="gripper_root_link">
+    <origin xyz="0.0 0.0 0.0" rpy="0.0 0.0 0.0"/>
+  </xacro:robotiq_85_gripper>
+  <!-- Sketch for conveyor -->
+  <link name="convayor_link">
+    <visual>
+      <geometry>
+        <box size="1.0 0.6 0.06"/>
+      </geometry>
+      <material name="green"/>
+    </visual>
+  </link>
+  <joint name="arm2convayor_joint" type="fixed">
+    <origin xyz="0.007 0.547 0.152" rpy="0 0 0"/>
+    <parent link="base_link"/>
+    <child link="convayor_link"/>
+  </joint>
+  <!-- TCP -->
+  <link name="tcp_link"/>
+  <joint name="gripper_base2tcp" type="fixed">
+    <parent link="robotiq_85_base_link"/>
+    <child link="tcp_link"/>
+    <origin xyz="0.13 0.0 0.0" rpy="0.0 0.0 0.0"/>
+  </joint>
 </robot>

Commit message: add coupler mesh

File: src/robot_description/urdf/system.urdf.xacro (robot description, xacro)
@@ -35,4 +35,18 @@
     <child link="camera_link"/>
   </joint>
+  <!-- Gripper coupler -->
+  <link name="gripper_coupler_link">
+    <visual>
+      <origin xyz="0.004 0.0 0.0" rpy="0.0 ${-M_PI/2} 0.0"/>
+      <geometry>
+        <mesh filename="package://robotiq_description/meshes/robotiq_85_coupler.stl"/>
+      </geometry>
+      <material name="black"/>
+    </visual>
+  </link>
+  <joint name="ee_link2coupler_joint" type="fixed">
+    <parent link="ee_link"/>
+    <child link="gripper_coupler_link"/>
+  </joint>
   <!-- Robotiq 2f 85 -->
   <link name="gripper_root_link"/>
@@ -62,5 +76,5 @@
   <link name="tcp_link"/>
   <joint name="gripper_base2tcp" type="fixed">
-    <parent link="robotiq_85_base_link"/>
+    <parent link="ee_link"/>
     <child link="tcp_link"/>
     <origin xyz="0.13 0.0 0.0" rpy="0.0 0.0 0.0"/>

Commit message: revise ee to tcp length

File: src/robot_description/urdf/system.urdf.xacro (robot description, xacro)
@@ -78,5 +78,5 @@
     <parent link="ee_link"/>
     <child link="tcp_link"/>
-    <origin xyz="0.13 0.0 0.0" rpy="0.0 0.0 0.0"/>
+    <origin xyz="0.15 0.0 0.0" rpy="0.0 0.0 0.0"/>
   </joint>
 </robot>

Commit message: add cam2 templete

File: src/robot_description/urdf/system.urdf.xacro (robot description, xacro)
@@ -19,6 +19,6 @@
   </material>
   <xacro:ur3_robot prefix="" joint_limited="false"/>
-  <!-- SR300 -->
-  <link name="camera_link">
+  <!-- SR300 above conveyor -->
+  <link name="camera1_link">
     <visual>
       <origin xyz="0.0 0.0 0.0" rpy="${M_PI/2} 0.0 ${M_PI/2}"/>
@@ -29,9 +29,24 @@
     </visual>
   </link>
-  <joint name="arm2cam_joint" type="fixed">
+  <joint name="arm2cam1_joint" type="fixed">
     <origin xyz="-0.0141949 0.45256924 0.84557343"
             rpy="2.8739904737308226 1.3575028048452842 1.3385069136920331"/>
     <parent link="base_link"/>
-    <child link="camera_link"/>
+    <child link="camera1_link"/>
+  </joint>
+  <!-- SR300 toward UR3 -->
+  <link name="camera2_link">
+    <visual>
+      <origin xyz="0.0 0.0 0.0" rpy="${M_PI/2} 0.0 ${M_PI/2}"/>
+      <geometry>
+        <mesh filename="package://realsense2_camera/meshes/RealSense 90deg.STL" scale="0.001 0.001 0.001"/>
+      </geometry>
+      <material name="black"/>
+    </visual>
+  </link>
+  <joint name="arm2cam2_joint" type="fixed">
+    <origin xyz="0 1.0 0.3" rpy="0.0 0.0 -${M_PI/2}"/> <!-- TBD -->
+    <parent link="base_link"/>
+    <child link="camera2_link"/>
   </joint>
   <!-- Gripper coupler -->

Commit message: revise spatial parameters

File: src/robot_description/urdf/system.urdf.xacro (robot description, xacro)
@@ -30,6 +30,6 @@
   </link>
   <joint name="arm2cam1_joint" type="fixed">
-    <origin xyz="-0.0141949 0.45256924 0.84557343"
-            rpy="2.8739904737308226 1.3575028048452842 1.3385069136920331"/>
+    <origin xyz="-0.00129317 0.440264 0.843718"
+            rpy="2.53724 1.54933 0.982746"/>
     <parent link="base_link"/>
     <child link="camera1_link"/>
@@ -46,5 +46,5 @@
   </link>
   <joint name="arm2cam2_joint" type="fixed">
-    <origin xyz="0 1.0 0.3" rpy="0.0 0.0 -${M_PI/2}"/> <!-- TBD -->
+    <origin xyz="-0.0368148 0.966091 0.409279" rpy="0.016628 0.132712 -1.55129"/> <!-- TBD -->
     <parent link="base_link"/>
     <child link="camera2_link"/>

Commit message: add suction system

File: src/robot_description/urdf/system.urdf.xacro (robot description, xacro)
@@ -8,7 +8,9 @@
   <xacro:property name="M_PI" value="3.1415926535"/>
   <!-- UR3 -->
-  <xacro:include filename="$(find ur_description)/urdf/ur3.urdf.xacro"/>
+  <!--xacro:include filename="$(find ur_description)/urdf/ur3.urdf.xacro"/-->
+  <!-- UR3 with suction -->
+  <xacro:include filename="$(find robot_description)/urdf/ur3_with_suction.urdf.xacro"/>
   <!-- Gripper -->
-  <xacro:include filename="$(find robotiq_description)/urdf/robotiq_85_gripper.urdf.xacro" />
+  <!--xacro:include filename="$(find robotiq_description)/urdf/robotiq_85_gripper.urdf.xacro" /-->
   <!-- Color material -->
   <material name="black">
@@ -51,4 +53,5 @@
   </joint>
   <!-- Gripper coupler -->
+  <!--
   <link name="gripper_coupler_link">
     <visual>
@@ -64,5 +67,4 @@
     <child link="gripper_coupler_link"/>
   </joint>
-  <!-- Robotiq 2f 85 -->
   <link name="gripper_root_link"/>
   <joint name="ee2gripper_joint" type="fixed">
@@ -74,4 +76,5 @@
     <origin xyz="0.0 0.0 0.0" rpy="0.0 0.0 0.0"/>
   </xacro:robotiq_85_gripper>
+  -->
   <!-- Sketch for conveyor -->
   <link name="convayor_link">
@@ -89,9 +92,9 @@
   </joint>
   <!-- TCP -->
-  <link name="tcp_link"/>
+  <!--link name="tcp_link"/>
   <joint name="gripper_base2tcp" type="fixed">
     <parent link="ee_link"/>
     <child link="tcp_link"/>
     <origin xyz="0.15 0.0 0.0" rpy="0.0 0.0 0.0"/>
-  </joint>
+  </joint-->
 </robot>

Commit message: recalibrate, revise tcp length

File: src/robot_description/urdf/system.urdf.xacro (robot description, xacro)
@@ -32,6 +32,6 @@
   </link>
   <joint name="arm2cam1_joint" type="fixed">
-    <origin xyz="-0.00129317 0.440264 0.843718"
-            rpy="2.53724 1.54933 0.982746"/>
+    <origin xyz="-0.00847729 0.45376 0.846709"
+            rpy="2.21937 1.55742 0.659318"/>
     <parent link="base_link"/>
     <child link="camera1_link"/>
@@ -92,9 +92,9 @@
   </joint>
   <!-- TCP -->
-  <!--link name="tcp_link"/>
+  <link name="tcp_link"/>
   <joint name="gripper_base2tcp" type="fixed">
     <parent link="ee_link"/>
     <child link="tcp_link"/>
-    <origin xyz="0.15 0.0 0.0" rpy="0.0 0.0 0.0"/>
-  </joint-->
+    <origin xyz="0.225 0.0 0.0" rpy="0.0 0.0 0.0"/>
+  </joint>
 </robot>

Commit message: revise parameter

File: src/robot_description/urdf/system.urdf.xacro (robot description, xacro)
@@ -32,11 +32,11 @@
   </link>
   <joint name="arm2cam1_joint" type="fixed">
-    <origin xyz="-0.00847729 0.45376 0.846709"
-            rpy="2.21937 1.55742 0.659318"/>
+    <origin xyz="-0.0247218 0.452686 0.852129"
+            rpy="2.70374 1.55653 1.12336"/>
     <parent link="base_link"/>
     <child link="camera1_link"/>
   </joint>
   <!-- SR300 toward UR3 -->
-  <link name="camera2_link">
+  <!--link name="camera2_link">
     <visual>
       <origin xyz="0.0 0.0 0.0" rpy="${M_PI/2} 0.0 ${M_PI/2}"/>
@@ -48,8 +48,8 @@
   </link>
   <joint name="arm2cam2_joint" type="fixed">
-    <origin xyz="-0.0368148 0.966091 0.409279" rpy="0.016628 0.132712 -1.55129"/> <!-- TBD -->
+    <origin xyz="-0.0368148 0.966091 0.409279" rpy="0.016628 0.132712 -1.55129"/>
     <parent link="base_link"/>
     <child link="camera2_link"/>
-  </joint>
+  </joint-->
   <!-- Gripper coupler -->
   <!--
@@ -96,5 +96,5 @@
     <parent link="ee_link"/>
     <child link="tcp_link"/>
-    <origin xyz="0.225 0.0 0.0" rpy="0.0 0.0 0.0"/>
+    <origin xyz="0.0 0.0 0.19" rpy="0.0 0.0 0.0"/>
   </joint>
 </robot>

Commit message: fix gripper tool from z to x axis

File: src/robot_description/urdf/system.urdf.xacro (robot description, xacro)
@@ -96,5 +96,5 @@
     <parent link="ee_link"/>
     <child link="tcp_link"/>
-    <origin xyz="0.0 0.0 0.19" rpy="0.0 0.0 0.0"/>
+    <origin xyz="0.19 0.0 0.0" rpy="0.0 0.0 0.0"/>
   </joint>
 </robot>

Commit message: change transformation for cam1, remove conveyor

File: src/robot_description/urdf/system.urdf.xacro (robot description, xacro)
@@ -32,6 +32,6 @@
   </link>
   <joint name="arm2cam1_joint" type="fixed">
-    <origin xyz="-0.0247218 0.452686 0.852129"
-            rpy="2.70374 1.55653 1.12336"/>
+    <origin xyz="-0.438475 -0.00906225 0.649185"
+            rpy="-2.65823 1.51606 -2.62462"/>
     <parent link="base_link"/>
     <child link="camera1_link"/>
@@ -77,24 +77,3 @@
   </xacro:robotiq_85_gripper>
   -->
-  <!-- Sketch for conveyor -->
-  <link name="convayor_link">
-    <visual>
-      <geometry>
-        <box size="1.0 0.6 0.06"/>
-      </geometry>
-      <material name="green"/>
-    </visual>
-  </link>
-  <joint name="arm2convayor_joint" type="fixed">
-    <origin xyz="0.007 0.547 0.152" rpy="0 0 0"/>
-    <parent link="base_link"/>
-    <child link="convayor_link"/>
-  </joint>
-  <!-- TCP -->
-  <link name="tcp_link"/>
-  <joint name="gripper_base2tcp" type="fixed">
-    <parent link="ee_link"/>
-    <child link="tcp_link"/>
-    <origin xyz="0.19 0.0 0.0" rpy="0.0 0.0 0.0"/>
-  </joint>
 </robot>

Commit message: change service, revise camera pose

File: src/robot_description/urdf/system.urdf.xacro (robot description, xacro)
@@ -32,6 +32,6 @@
   </link>
   <joint name="arm2cam1_joint" type="fixed">
-    <origin xyz="-0.438475 -0.00906225 0.649185"
-            rpy="-2.65823 1.51606 -2.62462"/>
+    <origin xyz="-0.662193 0.0253357 0.618725"
+            rpy="-0.212 1.192 -0.238"/>
     <parent link="base_link"/>
     <child link="camera1_link"/>

Commit message: recalibrated

File: src/robot_description/urdf/system.urdf.xacro (robot description, xacro)
@@ -32,6 +32,6 @@
   </link>
   <joint name="arm2cam1_joint" type="fixed">
-    <origin xyz="-0.662193 0.0253357 0.618725"
-            rpy="-0.212 1.192 -0.238"/>
+    <origin xyz="-0.731354 -0.0532628 0.600809"
+            rpy="0.056 1.138 0.060"/>
     <parent link="base_link"/>
     <child link="camera1_link"/>

Commit message: new config.

File: src/robot_description/urdf/system.urdf.xacro (robot description, xacro)
@@ -32,6 +32,6 @@
   </link>
   <joint name="arm2cam1_joint" type="fixed">
-    <origin xyz="-0.731354 -0.0532628 0.600809"
-            rpy="0.056 1.138 0.060"/>
+    <origin xyz="-0.685 -0.036 0.726"
+            rpy="0.053 1.242 0.085"/>
     <parent link="base_link"/>
     <child link="camera1_link"/>

Commit message: update extrinsic

File: src/robot_description/urdf/system.urdf.xacro (robot description, xacro)
@@ -32,6 +32,6 @@
   </link>
   <joint name="arm2cam1_joint" type="fixed">
-    <origin xyz="-0.685 -0.036 0.726"
-            rpy="0.053 1.242 0.085"/>
+    <origin xyz="-0.687477 -0.052075 0.723515"
+            rpy="0.170969 1.276745 0.220759"/>
     <parent link="base_link"/>
     <child link="camera1_link"/>

Commit message: update some configs

File: src/robot_description/urdf/system.urdf.xacro (robot description, xacro)
@@ -32,6 +32,6 @@
   </link>
   <joint name="arm2cam1_joint" type="fixed">
-    <origin xyz="-0.687477 -0.052075 0.723515"
-            rpy="0.170969 1.276745 0.220759"/>
+    <origin xyz="-0.673540 -0.035113 0.726538"
+            rpy="0.049012 1.178053 0.051708"/>
     <parent link="base_link"/>
     <child link="camera1_link"/>

Commit message: for ict demo

File: src/robot_description/urdf/system.urdf.xacro (robot description, xacro)
@@ -31,7 +31,16 @@
     </visual>
   </link>
+  <!-- For original version
   <joint name="arm2cam1_joint" type="fixed">
     <origin xyz="-0.673540 -0.035113 0.726538"
             rpy="0.049012 1.178053 0.051708"/>
+    <parent link="base_link"/>
+    <child link="camera1_link"/>
+  </joint>
+  !-->
+  <!-- For ICT demo -->
+  <joint name="arm2cam1_joint" type="fixed">
+    <origin xyz="-0.756954 -0.049132 0.930176"
+            rpy="0.018308 1.142433 0.030754"/>
     <parent link="base_link"/>
     <child link="camera1_link"/>

Commit message: shorten camera height

File: src/robot_description/urdf/system.urdf.xacro (robot description, xacro)
@@ -41,6 +41,6 @@
   <!-- For ICT demo -->
   <joint name="arm2cam1_joint" type="fixed">
-    <origin xyz="-0.756954 -0.049132 0.930176"
-            rpy="0.018308 1.142433 0.030754"/>
+    <origin xyz="-0.755580 -0.054556 0.784186"
+            rpy="0.047026 1.137168 0.063290"/>
     <parent link="base_link"/>
     <child link="camera1_link"/>
