Commit message: raise to prevent collision with ground

File: src/universal_robot/ur_description/urdf/ur3_robot.urdf.xacro (robot description, xacro)
@@ -13,5 +13,5 @@
     <parent link="world" />
     <child link = "base_link" />
-    <origin xyz="0.0 0.0 0.0" rpy="0.0 0.0 0.0" />
+    <origin xyz="0.0 0.0 2.0" rpy="0.0 0.0 0.0" />
   </joint>
 </robot>

File: src/universal_robot/ur_description/urdf/ur5_robot.urdf.xacro (robot description, xacro)
@@ -15,5 +15,5 @@
     <parent link="world" />
     <child link = "base_link" />
-    <origin xyz="0.0 0.0 0.0" rpy="0.0 0.0 0.0" />
+    <origin xyz="0.0 0.0 1.0" rpy="0.0 0.0 0.0" />
   </joint>
 </robot>
